Commit message: Updated xacro macro for tib block tool frame.

File: urdf/tib_mount/tib_tool_frame_macro.xacro (robot description, xacro)
@@ -1,5 +1,6 @@
 <?xml version="1.0"?>
 <robot xmlns:xacro="http://wiki.ros.org/xacro">
-    <xacro:macro name="Tool_Frame" params="prefix">
+    <xacro:include filename="$(find fanuc_resources)/urdf/common_materials.xacro"/>
+    <xacro:macro name="tib_tool" params="prefix">
         <xacro:property name="tool_mesh" value=
         "package://fanuc_m20ia_tools/meshes/tools/GL1807608_TibiaFibula_L_Reflected_Block_ROSI_Tib_Ref.stl" />
